File: MQ-135_Matheus_Rossetti_-_14205347.brd (EAGLE design)
At the start: 54.2 x 66.5 mm, 48 parts, among them J1 TP4056, Q1 500mA/300V, X1 FIDUCIAL_0.6-1.2MM, X2 5032, X3 FIDUCIAL_0.6-1.2MM

Commit message: 1.08052021.2336
Connections:
- removed net N$29: NUCLEO_STM32.18, R2.1, U$1.A$2, U$1.B$2
- removed net RX: BT_SENSOR.2, NUCLEO_STM32.27
- removed net TX: BT_SENSOR.1, NUCLEO_STM32.28
- new net ENTRADASENSOR: NUCLEO_STM32.15, R2.1, U$1.A$2, U$1.B$2
- new net N$21: BT_SENSOR.1, NUCLEO_STM32.29
- new net N$6: BT_SENSOR.2, NUCLEO_STM32.30
- net N$12: now also NUCLEO_STM32.20; no longer NUCLEO_STM32.10
- net N$15: now also NUCLEO_STM32.19; no longer NUCLEO_STM32.9
Routing:
- net ENTRADASENSOR: track 0.00 -> 30.7 mm
- net N$21: track 0.00 -> 29.9 mm
- net TX: track 29.2 -> 0.00 mm
- net RX: track 28.3 -> 0.00 mm
- net N$6: track 0.00 -> 27.1 mm, vias 0 -> 2
- net N$29: track 27.0 -> 0.00 mm
- net N$15: track 13.8 -> 21.5 mm, vias 0 -> 2
- net N$12: track 13.1 -> 20.6 mm, vias 0 -> 2
- net 3,3V: track 116.8 -> 111.7 mm, vias 5 -> 7
- net GND: track 268.6 -> 270.2 mm
