File: MQ-135_Matheus_Rossetti_-_14205347.sch (EAGLE design)
At the start: 48 parts, among them J1 TP4056, Q1 500mA/300V, X1 FIDUCIAL_0.6-1.2MM, X2 5032, X3 FIDUCIAL_0.6-1.2MM

Commit message: 1.08052021.2336
Connections:
- removed net N$29: NUCLEO_STM32.PA8, R2.1, U$1.A$2, U$1.B$2
- removed net RX: BT_SENSOR.UART_RX, NUCLEO_STM32.PB4
- removed net TX: BT_SENSOR.UART_TX, NUCLEO_STM32.PB5
- new net ENTRADASENSOR: NUCLEO_STM32.PB1, R2.1, U$1.A$2, U$1.B$2
- new net N$21: BT_SENSOR.UART_TX, NUCLEO_STM32.PB6
- new net N$6: BT_SENSOR.UART_RX, NUCLEO_STM32.PB7
- net N$12: now also NUCLEO_STM32.PA10; no longer NUCLEO_STM32.PA4
- net N$15: now also NUCLEO_STM32.PA9; no longer NUCLEO_STM32.PA3
Changed lines of the file:
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@@
 <setting verticaltext="up"/>
 </settings>
-<grid distance="0.1" unitdist="mm" unit="mm" style="lines" multiple="1" display="yes" altdistance="0.1" altunitdist="mm" altunit="mm"/>
+<grid distance="0.1" unitdist="mm" unit="mm" style="lines" multiple="1" display="no" altdistance="0.1" altunitdist="mm" altunit="mm"/>
 <layers>
 <layer number="1" name="Top" color="4" fill="1" visible="no" active="no"/>
@@
 <net name="N$12" class="0">
 <segment>
-<pinref part="NUCLEO_STM32" gate="G$1" pin="PA4"/>
-<wire x1="144.44" y1="170.76" x2="138" y2="170.76" width="0.1524" layer="91"/>
-<wire x1="138" y1="170.76" x2="138" y2="215" width="0.1524" layer="91"/>
 <pinref part="J3" gate="G$1" pin="2"/>
+<wire x1="138" y1="177.2" x2="138" y2="215" width="0.1524" layer="91"/>
 <wire x1="205.92" y1="215" x2="138" y2="215" width="0.1524" layer="91"/>
+<pinref part="NUCLEO_STM32" gate="G$1" pin="PA10"/>
+<wire x1="157.14" y1="142.82" x2="157.14" y2="177.2" width="0.1524" layer="91"/>
+<wire x1="157.14" y1="177.2" x2="138" y2="177.2" width="0.1524" layer="91"/>
 </segment>
 </net>
 <net name="N$15" class="0">
 <segment>
-<pinref part="NUCLEO_STM32" gate="G$1" pin="PA3"/>
-<wire x1="144.44" y1="173.3" x2="139" y2="173.3" width="0.1524" layer="91"/>
-<wire x1="139" y1="173.3" x2="139" y2="212.46" width="0.1524" layer="91"/>
 <pinref part="J3" gate="G$1" pin="3"/>
+<wire x1="139" y1="179.3" x2="139" y2="212.46" width="0.1524" layer="91"/>
 <wire x1="205.92" y1="212.46" x2="139" y2="212.46" width="0.1524" layer="91"/>
+<pinref part="NUCLEO_STM32" gate="G$1" pin="PA9"/>
+<wire x1="159.68" y1="142.82" x2="159.68" y2="179.3" width="0.1524" layer="91"/>
+<wire x1="159.68" y1="179.3" x2="139" y2="179.3" width="0.1524" layer="91"/>
 </segment>
 </net>
@@
 </segment>
 </net>
-<net name="N$29" class="0">
+<net name="ENTRADASENSOR" class="0">
 <segment>
 <pinref part="U$1" gate="G$1" pin="B$2"/>
@@
 <wire x1="231" y1="198" x2="225.08" y2="198" width="0.1524" layer="91"/>
 <wire x1="231" y1="198" x2="231" y2="139" width="0.1524" layer="91"/>
-<wire x1="231" y1="139" x2="164.76" y2="139" width="0.1524" layer="91"/>
-<pinref part="NUCLEO_STM32" gate="G$1" pin="PA8"/>
-<wire x1="164.76" y1="139" x2="164.76" y2="142.82" width="0.1524" layer="91"/>
+<wire x1="231" y1="139" x2="164.8" y2="139" width="0.1524" layer="91"/>
+<wire x1="164.8" y1="139" x2="164.76" y2="139" width="0.1524" layer="91"/>
+<wire x1="164.8" y1="139" x2="164.8" y2="129.3" width="0.1524" layer="91"/>
+<junction x="164.8" y="139"/>
+<wire x1="164.8" y1="129.3" x2="132" y2="129.3" width="0.1524" layer="91"/>
+<wire x1="132" y1="129.3" x2="132" y2="158.06" width="0.1524" layer="91"/>
+<pinref part="NUCLEO_STM32" gate="G$1" pin="PB1"/>
+<wire x1="132" y1="158.06" x2="144.44" y2="158.06" width="0.1524" layer="91"/>
 </segment>
 </net>
@@
 <wire x1="101" y1="251.38" x2="100.56" y2="251.38" width="0.1524" layer="91"/>
 <junction x="100.56" y="251.38"/>
-</segment>
-</net>
-<net name="TX" class="0">
-<segment>
-<pinref part="NUCLEO_STM32" gate="G$1" pin="PB5"/>
-<pinref part="BT_SENSOR" gate="G$1" pin="UART_TX"/>
-<wire x1="197.78" y1="163.14" x2="235.92" y2="163.14" width="0.1524" layer="91"/>
-<wire x1="235.92" y1="163.14" x2="235.92" y2="164.84" width="0.1524" layer="91"/>
-</segment>
-</net>
-<net name="RX" class="0">
-<segment>
-<pinref part="NUCLEO_STM32" gate="G$1" pin="PB4"/>
-<pinref part="BT_SENSOR" gate="G$1" pin="UART_RX"/>
-<wire x1="197.78" y1="160.6" x2="235.92" y2="160.6" width="0.1524" layer="91"/>
-<wire x1="235.92" y1="160.6" x2="235.92" y2="162.3" width="0.1524" layer="91"/>
 </segment>
 </net>
@@
 </segment>
 </net>
+<net name="N$6" class="0">
+<segment>
+<pinref part="BT_SENSOR" gate="G$1" pin="UART_RX"/>
+<wire x1="235.92" y1="162.3" x2="235.92" y2="162.56" width="0.1524" layer="91"/>
+<wire x1="235.92" y1="162.56" x2="200.66" y2="162.56" width="0.1524" layer="91"/>
+<wire x1="200.66" y1="162.56" x2="200.66" y2="168.22" width="0.1524" layer="91"/>
+<pinref part="NUCLEO_STM32" gate="G$1" pin="PB7"/>
+<wire x1="200.66" y1="168.22" x2="197.78" y2="168.22" width="0.1524" layer="91"/>
+</segment>
+</net>
+<net name="N$21" class="0">
+<segment>
+<pinref part="NUCLEO_STM32" gate="G$1" pin="PB6"/>
+<wire x1="197.78" y1="158.06" x2="228.6" y2="158.06" width="0.1524" layer="91"/>
+<wire x1="228.6" y1="158.06" x2="228.6" y2="165.1" width="0.1524" layer="91"/>
+<pinref part="BT_SENSOR" gate="G$1" pin="UART_TX"/>
+<wire x1="228.6" y1="165.1" x2="235.92" y2="165.1" width="0.1524" layer="91"/>
+<wire x1="235.92" y1="165.1" x2="235.92" y2="164.84" width="0.1524" layer="91"/>
+</segment>
+</net>
